Commit message: updating urdf and key control cart file

File: lfd-omnid-algorithm/src/cartpole_gazebo/urdf/carpole_gazebo_urdf.xacro.urdf (robot description, URDF)
Before this commit: robot cartopole, 5 links, 4 joints
Links:
- link box: mass 3 -> 15
- link cart: mass 5 -> 20
- link pole: geometry visual box size=0.05 0.05 1.5
Joints:
- joint pole_to_box: origin xyz=0.0 0.0 -1.0 -> xyz=0.0 0.0 -1.5

Commit message: Changing ros simulation files

File: lfd-omnid-algorithm/src/cartpole_gazebo/urdf/carpole_gazebo_urdf.xacro.urdf (robot description, URDF)
Before this commit: robot cartopole, 5 links, 4 joints
Links:
- removed link box
- link pole: mass 10 -> 20; geometry visual box size=0.05 0.05 2.0
Joints:
- removed joint pole_to_box
